File: IP6557_Charger.kicad_pcb (KiCad board)
At the start: 4 copper layers, 38.5 x 14.7 mm, 44 parts, among them J1 Conn_01x04, J2 XKB_U262-16XN, Q1 CSD17581Q3A, Q2 CSD17581Q3A, Q3 CSD17581Q3A, Q4 CSD17581Q3A, U1 IP6557_C, U2 ESD224DQA

Commit message: Upd
Parts:
- added C19: 22uF, Capacitor_SMD:C_0805_2012Metric, B.Cu at (113.2, 112.9)
- added C21: 22uF, Capacitor_SMD:C_0805_2012Metric, B.Cu at (111.2, 112.9)
- added C22: 22uF, Capacitor_SMD:C_0805_2012Metric, B.Cu at (109.2, 112.9)
- added C25: 1uF, Capacitor_SMD:C_0603_1608Metric, B.Cu at (106.7, 109.1)
- added C27: 100nF, Capacitor_SMD:C_0402_1005Metric, B.Cu at (124.2, 100.7)
- added C4: 100uF, IP6557_Charger:CP_Radial_D5.0mm_P2.00mm, F.Cu at (109.4, 111.0)
- added C7: 470uF, IP6557_Charger:CP_Radial_D8.0mm_P3.50mm, F.Cu at (130.0, 105.6)
- added C8: 1uF, Capacitor_SMD:C_0805_2012Metric, B.Cu at (132.9, 113.5)
- added D1: SMF36A, Diode_SMD:D_SMF, F.Cu at (102.2, 113.4)
- C1: renamed from C4; value 100uF -> 10uF
- C2: renamed from C8; value 100uF -> 10uF
- C3: renamed from C6; value 100uF -> 10uF
- F1: footprint Fuse:Fuse_0805_2012Metric -> Fuse:Fuse_1206_3216Metric
- moved R3 4.05 mm to (118.5, 111.0)
- moved C18 3.96 mm to (118.5, 110.0)
- moved R4 0.88 mm to (118.0, 103.8)
- moved C26 0.75 mm to (106.8, 110.8)
- moved C10 0.36 mm to (127.9, 100.7)
- moved C11 0.09 mm to (126.1, 100.7)
- renumbered C16 to C10, C15 to C11, C20 to C12, C11 to C13, C13 to C14, C22 to C15, C12 to C16, C14 to C17, C17 to C18, C10 to C20, C3 to C23, C2 to C24, C1 to C26, C18 to C5, C19 to C6, C21 to C9, D1 to D2, D2 to D3, D3 to D4, D4 to D5, Q4 to Q1, Q3 to Q2, Q1 to Q3, Q2 to Q4, R5 to R1, R1 to R10, R6 to R2, R9 to R3, R8 to R4, R7 to R5, R10 to R6, R2 to R7, R3 to R8, R4 to R9, U2 to U1, U1 to U2
Routing:
- net Net-(U2-CSP_{1}): track 13.5 -> 8.86 mm, vias 2 -> 0
- net /PCON: track 16.6 -> 13.2 mm, vias 2 -> 0
- net Net-(U2-CSN_{1}): track 21.7 -> 18.6 mm, vias 11 -> 30
- net /CC2_{1}: track 6.40 -> 8.66 mm
- net /CSP2: track 48.0 -> 49.1 mm, vias 1 -> 29
- net /LG1: track 6.39 -> 5.64 mm
- net GND: vias 1 -> 73
- added copper zone on F.Cu, net /CSP2
Other:
- outline, holes or cut-outs redrawn
- board text added: "Designed by Acha-${CURRENT_DATE}"
- board text added: "IP6557_Charger ${BRANCH}-${SHORT_SHA}"

Commit message: Upd
Routing:
- net /DP_{1}: track 8.26 -> 7.27 mm
- net /CC1_{1}: track 6.64 -> 5.98 mm
- net /PCIN: track 23.7 -> 23.0 mm
- net /PCON: track 13.2 -> 12.7 mm
- net GND: vias 73 -> 77

Commit message: Upd
Parts:
- Q1, Q2, Q3, Q4: value CSD17581Q3A -> NTTFS5C673NL
